Commit message: finished task a.2

File: nuturtle_description/urdf/turtlebot3_burger.urdf.xacro (robot description, xacro)
@@ -1,10 +1,44 @@
+<?xml version="1.0" ?>
 <!-- Note that this file has been modified by Ayush Gaggar on Jan. 10. 2023
      for the purposes of a class assignment. The rights of the original source code
      can be found on the github of robotis' turtlebot3 repo. The changes made to the
      original file are largely aesthetic changes made for educational purposes. -->
-<?xml version="1.0" ?>
 <robot name="turtlebot3_burger" xmlns:xacro="http://ros.org/wiki/xacro">
-  <xacro:include filename="$(find turtlebot3_description)/urdf/common_properties.xacro"/>
-  <xacro:include filename="$(find turtlebot3_description)/urdf/turtlebot3_burger.gazebo.xacro"/>
+  <!-- <xacro:include filename="$(find turtlebot3_description)/urdf/common_properties.urdf"/> -->
+  <!-- <xacro:include filename="$(find nuturtle_description)/meshes/burger_base.stl"/>
+  <xacro:include filename="$(find nuturtle_description)/meshes/lds.stl"/>
+  <xacro:include filename="$(find nuturtle_description)/meshes/left_tire.stl"/>
+  <xacro:include filename="$(find nuturtle_description)/meshes/right_tire.stl"/> -->
+  <!-- Init colour -->
+  <material name="black">
+      <color rgba="0.0 0.0 0.0 1.0"/>
+  </material>
+  <material name="dark">
+    <color rgba="0.3 0.3 0.3 1.0"/>
+  </material>
+  <material name="light_black">
+    <color rgba="0.4 0.4 0.4 1.0"/>
+  </material>
+  <material name="blue">
+    <color rgba="0.0 0.0 0.8 1.0"/>
+  </material>
+  <material name="green">
+    <color rgba="0.0 0.8 0.0 1.0"/>
+  </material>
+  <material name="grey">
+    <color rgba="0.5 0.5 0.5 1.0"/>
+  </material>
+  <material name="orange">
+    <color rgba="1.0 0.4235 0.0392 1.0"/>
+  </material>
+  <material name="brown">
+    <color rgba="0.8706 0.8118 0.7647 1.0"/>
+  </material>
+  <material name="red">
+    <color rgba="0.8 0.0 0.0 1.0"/>
+  </material>
+  <material name="white">
+    <color rgba="1.0 1.0 1.0 1.0"/>
+  </material>
   <link name="base_footprint"/>
   <joint name="base_joint" type="fixed">
@@ -17,5 +51,5 @@
       <origin xyz="-0.032 0 0.0" rpy="0 0 0"/>
       <geometry>
-        <mesh filename="package://turtlebot3_description/meshes/bases/burger_base.stl" scale="0.001 0.001 0.001"/>
+        <mesh filename="package://nuturtle_description/meshes/burger_base.stl" scale="0.001 0.001 0.001"/>
       </geometry>
       <material name="light_black"/>
@@ -30,7 +64,5 @@
       <origin xyz="0 0 0" rpy="0 0 0"/>
       <mass value="8.2573504e-01"/>
-      <inertia ixx="2.2124416e-03" ixy="-1.2294101e-05" ixz="3.4938785e-05"
-               iyy="2.1193702e-03" iyz="-5.0120904e-06"
-               izz="2.0064271e-03" />
+      <inertia ixx="2.2124416e-03" ixy="-1.2294101e-05" ixz="3.4938785e-05" iyy="2.1193702e-03" iyz="-5.0120904e-06" izz="2.0064271e-03" />
     </inertial>
   </link>
@@ -45,5 +77,5 @@
       <origin xyz="0 0 0" rpy="1.57 0 0"/>
       <geometry>
-        <mesh filename="package://turtlebot3_description/meshes/wheels/left_tire.stl" scale="0.001 0.001 0.001"/>
+        <mesh filename="package://nuturtle_description/meshes/left_tire.stl" scale="0.001 0.001 0.001"/>
       </geometry>
       <material name="dark"/>
@@ -58,8 +90,6 @@
       <origin xyz="0 0 0" />
       <mass value="2.8498940e-02" />
-      <inertia ixx="1.1175580e-05" ixy="-4.2369783e-11" ixz="-5.9381719e-09"
-               iyy="1.1192413e-05" iyz="-1.4400107e-11"
-               izz="2.0712558e-05" />
-      </inertial>
+      <inertia ixx="1.1175580e-05" ixy="-4.2369783e-11" ixz="-5.9381719e-09" iyy="1.1192413e-05" iyz="-1.4400107e-11" izz="2.0712558e-05" />
+    </inertial>
   </link>
   <joint name="wheel_right_joint" type="continuous">
@@ -73,5 +103,5 @@
       <origin xyz="0 0 0" rpy="1.57 0 0"/>
       <geometry>
-        <mesh filename="package://turtlebot3_description/meshes/wheels/right_tire.stl" scale="0.001 0.001 0.001"/>
+        <mesh filename="package://nuturtle_description/meshes/right_tire.stl" scale="0.001 0.001 0.001"/>
       </geometry>
       <material name="dark"/>
@@ -86,8 +116,6 @@
       <origin xyz="0 0 0" />
       <mass value="2.8498940e-02" />
-      <inertia ixx="1.1175580e-05" ixy="-4.2369783e-11" ixz="-5.9381719e-09"
-               iyy="1.1192413e-05" iyz="-1.4400107e-11"
-               izz="2.0712558e-05" />
-      </inertial>
+      <inertia ixx="1.1175580e-05" ixy="-4.2369783e-11" ixz="-5.9381719e-09" iyy="1.1192413e-05" iyz="-1.4400107e-11" izz="2.0712558e-05" />
+    </inertial>
   </link>
   <joint name="caster_back_joint" type="fixed">
@@ -106,7 +134,5 @@
       <origin xyz="0 0 0" />
       <mass value="0.005" />
-      <inertia ixx="0.001" ixy="0.0" ixz="0.0"
-               iyy="0.001" iyz="0.0"
-               izz="0.001" />
+      <inertia ixx="0.001" ixy="0.0" ixz="0.0" iyy="0.001" iyz="0.0" izz="0.001" />
     </inertial>
   </link>
@@ -126,5 +152,5 @@
       <origin xyz="0 0 0.0" rpy="0 0 0"/>
       <geometry>
-        <mesh filename="package://turtlebot3_description/meshes/sensors/lds.stl" scale="0.001 0.001 0.001"/>
+        <mesh filename="package://nuturtle_description/meshes/lds.stl" scale="0.001 0.001 0.001"/>
       </geometry>
       <material name="dark"/>
@@ -139,7 +165,5 @@
       <mass value="0.114" />
       <origin xyz="0 0 0" />
-      <inertia ixx="0.001" ixy="0.0" ixz="0.0"
-               iyy="0.001" iyz="0.0"
-               izz="0.001" />
+      <inertia ixx="0.001" ixy="0.0" ixz="0.0" iyy="0.001" iyz="0.0" izz="0.001" />
     </inertial>
   </link>

Commit message: finished task a3

File: nuturtle_description/urdf/turtlebot3_burger.urdf.xacro (robot description, xacro)
@@ -5,5 +5,14 @@
      original file are largely aesthetic changes made for educational purposes. -->
 <robot name="turtlebot3_burger" xmlns:xacro="http://ros.org/wiki/xacro">
-  <!-- <xacro:include filename="$(find turtlebot3_description)/urdf/common_properties.urdf"/> -->
+  <xacro:property name="yaml" value="$(find nuturtle_description)/config/diff_params.yaml" />
+  <xacro:property name="props" value="${xacro.load_yaml(yaml)}" />
+  <xacro:property name="ros_param" value="${props['/**']}" />
+  <xacro:property name="parameters" value="${ros_param['ros__parameters']}" />
+  <xacro:property name="wheel_radius" value="${parameters['wheel_radius']}" />
+  <xacro:property name="track_width" value="${parameters['track_width']}" />
+  <xacro:property name="motor_cmd_max" value="${parameters['motor_cmd_max']}" />
+  <xacro:property name="motor_cmd_per_rad_sec" value="${parameters['motor_cmd_per_rad_sec']}" />
+  <xacro:property name="encoder_ticks_per_rad" value="${parameters['encoder_ticks_per_rad']}" />
+  <xacro:property name="collision_radius" value="${parameters['collision_radius']}" />
   <!-- Init colour -->
   <material name="black">
@@ -54,5 +63,10 @@
       <origin xyz="-0.032 0 0.070" rpy="0 0 0"/>
       <geometry>
-        <box size="0.140 0.140 0.143"/>
+        <xacro:if value="${collision_radius &lt; 0.0}">
+          <box size="0.140 0.140 0.143"/>
+        </xacro:if>
+        <xacro:unless value="${collision_radius &gt; 0.0}">
+          <cylinder radius="0.140" length="0.143"/>
+        </xacro:unless>
       </geometry>
     </collision>
@@ -66,5 +80,5 @@
     <parent link="base_link"/>
     <child link="wheel_left_link"/>
-    <origin xyz="0.0 0.08 0.023" rpy="-1.57 0 0"/>
+    <origin xyz="0.0 ${track_width/2} 0.023" rpy="-1.57 0 0"/>
     <axis xyz="0 0 1"/>
   </joint>
@@ -80,5 +94,5 @@
       <origin xyz="0 0 0" rpy="0 0 0"/>
       <geometry>
-        <cylinder length="0.018" radius="0.033"/>
+        <cylinder length="0.018" radius="${wheel_radius}"/>
       </geometry>
     </collision>
@@ -92,5 +106,5 @@
     <parent link="base_link"/>
     <child link="wheel_right_link"/>
-    <origin xyz="0.0 -0.080 0.023" rpy="-1.57 0 0"/>
+    <origin xyz="0.0 -${track_width/2} 0.023" rpy="-1.57 0 0"/>
     <axis xyz="0 0 1"/>
   </joint>

Commit message: working on a.4

File: nuturtle_description/urdf/turtlebot3_burger.urdf.xacro (robot description, xacro)
@@ -15,4 +15,6 @@
   <xacro:property name="encoder_ticks_per_rad" value="${parameters['encoder_ticks_per_rad']}" />
   <xacro:property name="collision_radius" value="${parameters['collision_radius']}" />
+  <xacro:arg name="color" default="purple" />
+  <xacro:property name="color" value="$(arg color)" />
   <!-- Init colour -->
   <material name="black">
@@ -58,5 +60,18 @@
         <mesh filename="package://nuturtle_description/meshes/burger_base.stl" scale="0.001 0.001 0.001"/>
       </geometry>
-      <material name="light_black"/>
+      <xacro:if value="${color == purple}">
+        <material name="purple">
+          <color rgba="0.3 0.16 0.52 1.0"/>
+        </material>
+      </xacro:if>
+      <xacro:if value="${color == red}">
+        <material name="red" />
+      </xacro:if>
+      <xacro:if value="${color == blue}">
+        <material name="red" />
+      </xacro:if>
+      <xacro:if value="${color == green}">
+        <material name="red" />
+      </xacro:if>
     </visual>
     <collision>

Commit message: finished task a.4

File: nuturtle_description/urdf/turtlebot3_burger.urdf.xacro (robot description, xacro)
@@ -60,29 +60,31 @@
         <mesh filename="package://nuturtle_description/meshes/burger_base.stl" scale="0.001 0.001 0.001"/>
       </geometry>
-      <xacro:if value="${color == purple}">
+      <xacro:if value="${color == 'purple'}">
         <material name="purple">
           <color rgba="0.3 0.16 0.52 1.0"/>
         </material>
       </xacro:if>
-      <xacro:if value="${color == red}">
+      <xacro:if value="${color == 'red'}">
         <material name="red" />
       </xacro:if>
-      <xacro:if value="${color == blue}">
-        <material name="red" />
+      <xacro:if value="${color == 'blue'}">
+        <material name="blue" />
       </xacro:if>
-      <xacro:if value="${color == green}">
-        <material name="red" />
+      <xacro:if value="${color == 'green'}">
+        <material name="green" />
       </xacro:if>
     </visual>
     <collision>
       <origin xyz="-0.032 0 0.070" rpy="0 0 0"/>
-      <geometry>
-        <xacro:if value="${collision_radius &lt; 0.0}">
+      <xacro:if value="${collision_radius &lt; 0.0}">
+        <geometry>
           <box size="0.140 0.140 0.143"/>
-        </xacro:if>
-        <xacro:unless value="${collision_radius &gt; 0.0}">
+        </geometry>
+      </xacro:if>
+      <xacro:if value="${collision_radius &gt; 0.0}">
+        <geometry>
           <cylinder radius="0.140" length="0.143"/>
-        </xacro:unless>
-      </geometry>
+        </geometry>
+      </xacro:if>
     </collision>
     <inertial>
